File: kicad/nw12887.kicad_pcb (KiCad board)
At the start: 2 copper layers, 18.3 x 31.1 mm, 4 parts, among them U1 ds12887, U2 ds12887, Y1 Crystal_Small

Commit message: Updated parts names
Parts:
- renumbered U2 to U1, U1 to U2
Changed lines of the file:
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@@
     (add_net INT)
     (add_net MOT)
-    (add_net "Net-(U1-Pad16)")
-    (add_net "Net-(U1-Pad2)")
-    (add_net "Net-(U1-Pad20)")
     (add_net "Net-(U1-Pad21)")
     (add_net "Net-(U1-Pad22)")
-    (add_net "Net-(U1-Pad3)")
+    (add_net "Net-(U2-Pad16)")
+    (add_net "Net-(U2-Pad2)")
+    (add_net "Net-(U2-Pad20)")
     (add_net "Net-(U2-Pad21)")
     (add_net "Net-(U2-Pad22)")
+    (add_net "Net-(U2-Pad3)")
     (add_net RST)
     (add_net RW)
@@
     (descr "24-lead though-hole mounted DIP package, row spacing 15.24 mm (600 mils), Socket")
     (tags "THT DIP DIL PDIP 2.54mm 15.24mm 600mil Socket")
-    (fp_text reference U1 (at 7.62 -2.33) (layer F.SilkS) hide
+    (fp_text reference U2 (at 7.62 -2.33) (layer F.SilkS) hide
       (effects (font (size 1 1) (thickness 0.15)))
     )
@@
       (effects (font (size 1 1) (thickness 0.15)))
     )
+    (fp_line (start 16.8 -1.6) (end -1.55 -1.6) (layer F.CrtYd) (width 0.05))
+    (fp_line (start 16.8 29.55) (end 16.8 -1.6) (layer F.CrtYd) (width 0.05))
+    (fp_line (start -1.55 29.55) (end 16.8 29.55) (layer F.CrtYd) (width 0.05))
+    (fp_line (start -1.55 -1.6) (end -1.55 29.55) (layer F.CrtYd) (width 0.05))
+    (fp_line (start 16.51 -1.33) (end -1.27 -1.33) (layer F.Fab) (width 0.1))
+    (fp_line (start 16.51 29.27) (end 16.51 -1.33) (layer F.Fab) (width 0.1))
+    (fp_line (start -1.27 29.27) (end 16.51 29.27) (layer F.Fab) (width 0.1))
+    (fp_line (start -1.27 -1.33) (end -1.27 29.27) (layer F.Fab) (width 0.1))
+    (fp_line (start 0.255 -0.27) (end 1.255 -1.27) (layer F.Fab) (width 0.1))
+    (fp_line (start 0.255 29.21) (end 0.255 -0.27) (layer F.Fab) (width 0.1))
+    (fp_line (start 14.985 29.21) (end 0.255 29.21) (layer F.Fab) (width 0.1))
+    (fp_line (start 14.985 -1.27) (end 14.985 29.21) (layer F.Fab) (width 0.1))
+    (fp_line (start 1.255 -1.27) (end 14.985 -1.27) (layer F.Fab) (width 0.1))
     (fp_text user %R (at 7.62 13.97) (layer F.Fab) hide
       (effects (font (size 1 1) (thickness 0.15)))
     )
-    (fp_line (start 1.255 -1.27) (end 14.985 -1.27) (layer F.Fab) (width 0.1))
-    (fp_line (start 14.985 -1.27) (end 14.985 29.21) (layer F.Fab) (width 0.1))
-    (fp_line (start 14.985 29.21) (end 0.255 29.21) (layer F.Fab) (width 0.1))
-    (fp_line (start 0.255 29.21) (end 0.255 -0.27) (layer F.Fab) (width 0.1))
-    (fp_line (start 0.255 -0.27) (end 1.255 -1.27) (layer F.Fab) (width 0.1))
-    (fp_line (start -1.27 -1.33) (end -1.27 29.27) (layer F.Fab) (width 0.1))
-    (fp_line (start -1.27 29.27) (end 16.51 29.27) (layer F.Fab) (width 0.1))
-    (fp_line (start 16.51 29.27) (end 16.51 -1.33) (layer F.Fab) (width 0.1))
-    (fp_line (start 16.51 -1.33) (end -1.27 -1.33) (layer F.Fab) (width 0.1))
-    (fp_line (start -1.55 -1.6) (end -1.55 29.55) (layer F.CrtYd) (width 0.05))
-    (fp_line (start -1.55 29.55) (end 16.8 29.55) (layer F.CrtYd) (width 0.05))
-    (fp_line (start 16.8 29.55) (end 16.8 -1.6) (layer F.CrtYd) (width 0.05))
-    (fp_line (start 16.8 -1.6) (end -1.55 -1.6) (layer F.CrtYd) (width 0.05))
     (pad 24 thru_hole oval (at 15.24 0) (size 1.6 1.6) (drill 0.8) (layers *.Cu *.Mask)
       (net 2 VCC))
@@
     (tags "SSOP 0.635")
     (attr smd)
-    (fp_text reference U2 (at 0 5.4) (layer B.SilkS)
+    (fp_text reference U1 (at 0 5.4) (layer B.SilkS)
       (effects (font (size 1 1) (thickness 0.15)) (justify mirror))
     )
@@
       (effects (font (size 1 1) (thickness 0.15)) (justify mirror))
     )
+    (fp_line (start -2.075 4) (end -3.2 4) (layer B.SilkS) (width 0.15))
+    (fp_line (start -2.075 -4.475) (end 2.075 -4.475) (layer B.SilkS) (width 0.15))
+    (fp_line (start -2.075 4.475) (end 2.075 4.475) (layer B.SilkS) (width 0.15))
+    (fp_line (start -2.075 -4.475) (end -2.075 -3.9175) (layer B.SilkS) (width 0.15))
+    (fp_line (start 2.075 -4.475) (end 2.075 -3.9175) (layer B.SilkS) (width 0.15))
+    (fp_line (start 2.075 4.475) (end 2.075 3.9175) (layer B.SilkS) (width 0.15))
+    (fp_line (start -2.075 4.475) (end -2.075 4) (layer B.SilkS) (width 0.15))
+    (fp_line (start -3.45 -4.65) (end 3.45 -4.65) (layer B.CrtYd) (width 0.05))
+    (fp_line (start -3.45 4.65) (end 3.45 4.65) (layer B.CrtYd) (width 0.05))
+    (fp_line (start 3.45 4.65) (end 3.45 -4.65) (layer B.CrtYd) (width 0.05))
+    (fp_line (start -3.45 4.65) (end -3.45 -4.65) (layer B.CrtYd) (width 0.05))
+    (fp_line (start -1.95 3.35) (end -0.95 4.35) (layer B.Fab) (width 0.15))
+    (fp_line (start -1.95 -4.35) (end -1.95 3.35) (layer B.Fab) (width 0.15))
+    (fp_line (start 1.95 -4.35) (end -1.95 -4.35) (layer B.Fab) (width 0.15))
+    (fp_line (start 1.95 4.35) (end 1.95 -4.35) (layer B.Fab) (width 0.15))
     (fp_line (start -0.95 4.35) (end 1.95 4.35) (layer B.Fab) (width 0.15))
-    (fp_line (start 1.95 4.35) (end 1.95 -4.35) (layer B.Fab) (width 0.15))
-    (fp_line (start 1.95 -4.35) (end -1.95 -4.35) (layer B.Fab) (width 0.15))
-    (fp_line (start -1.95 -4.35) (end -1.95 3.35) (layer B.Fab) (width 0.15))
-    (fp_line (start -1.95 3.35) (end -0.95 4.35) (layer B.Fab) (width 0.15))
-    (fp_line (start -3.45 4.65) (end -3.45 -4.65) (layer B.CrtYd) (width 0.05))
-    (fp_line (start 3.45 4.65) (end 3.45 -4.65) (layer B.CrtYd) (width 0.05))
-    (fp_line (start -3.45 4.65) (end 3.45 4.65) (layer B.CrtYd) (width 0.05))
-    (fp_line (start -3.45 -4.65) (end 3.45 -4.65) (layer B.CrtYd) (width 0.05))
-    (fp_line (start -2.075 4.475) (end -2.075 4) (layer B.SilkS) (width 0.15))
-    (fp_line (start 2.075 4.475) (end 2.075 3.9175) (layer B.SilkS) (width 0.15))
-    (fp_line (start 2.075 -4.475) (end 2.075 -3.9175) (layer B.SilkS) (width 0.15))
-    (fp_line (start -2.075 -4.475) (end -2.075 -3.9175) (layer B.SilkS) (width 0.15))
-    (fp_line (start -2.075 4.475) (end 2.075 4.475) (layer B.SilkS) (width 0.15))
-    (fp_line (start -2.075 -4.475) (end 2.075 -4.475) (layer B.SilkS) (width 0.15))
-    (fp_line (start -2.075 4) (end -3.2 4) (layer B.SilkS) (width 0.15))
     (fp_text user %R (at 0 0) (layer B.Fab)
       (effects (font (size 0.8 0.8) (thickness 0.15)) (justify mirror))
@@
       (effects (font (size 1 1) (thickness 0.15)))
     )
+    (fp_line (start 5 7.9) (end 5 5.6) (layer F.SilkS) (width 0.12))
+    (fp_line (start -5 7.9) (end 5 7.9) (layer F.SilkS) (width 0.12))
+    (fp_line (start -5 5.6) (end -5 7.9) (layer F.SilkS) (width 0.12))
     (fp_circle (center 0 0) (end 0.1 -7.5) (layer F.SilkS) (width 0.12))
-    (fp_line (start -5 5.6) (end -5 7.9) (layer F.SilkS) (width 0.12))
-    (fp_line (start -5 7.9) (end 5 7.9) (layer F.SilkS) (width 0.12))
-    (fp_line (start 5 7.9) (end 5 5.6) (layer F.SilkS) (width 0.12))
     (pad 1 smd rect (at 0 8 180) (size 2.3 4) (layers F.Cu F.Paste F.Mask)
       (net 19 BC))
@@
       (effects (font (size 1 1) (thickness 0.15)) (justify mirror))
     )
+    (fp_line (start 2.1 4.63) (end -2.1 4.63) (layer B.CrtYd) (width 0.05))
+    (fp_line (start 2.1 -5.07) (end 2.1 4.63) (layer B.CrtYd) (width 0.05))
+    (fp_line (start -2.1 -5.07) (end 2.1 -5.07) (layer B.CrtYd) (width 0.05))
+    (fp_line (start -2.1 4.63) (end -2.1 -5.07) (layer B.CrtYd) (width 0.05))
+    (fp_line (start 1.27 2.5) (end 1.27 2.5) (layer B.SilkS) (width 0.12))
+    (fp_line (start 0.5 2.1) (end 1.27 2.5) (layer B.SilkS) (width 0.12))
+    (fp_line (start -1.27 2.5) (end -1.27 2.5) (layer B.SilkS) (width 0.12))
+    (fp_line (start -0.5 2.1) (end -1.27 2.5) (layer B.SilkS) (width 0.12))
+    (fp_line (start 1.7 2.1) (end -1.7 2.1) (layer B.SilkS) (width 0.12))
+    (fp_line (start 1.7 -4.5) (end 1.7 2.1) (layer B.SilkS) (width 0.12))
+    (fp_line (start -1.7 -4.5) (end 1.7 -4.5) (layer B.SilkS) (width 0.12))
+    (fp_line (start -1.7 2.1) (end -1.7 -4.5) (layer B.SilkS) (width 0.12))
+    (fp_line (start 1.27 2.7) (end 1.27 3.5) (layer B.Fab) (width 0.1))
+    (fp_line (start 0.5 1.9) (end 1.27 2.7) (layer B.Fab) (width 0.1))
+    (fp_line (start -1.27 2.7) (end -1.27 3.5) (layer B.Fab) (width 0.1))
+    (fp_line (start -0.5 1.9) (end -1.27 2.7) (layer B.Fab) (width 0.1))
+    (fp_line (start 0.95 1.9) (end -0.95 1.9) (layer B.Fab) (width 0.1))
+    (fp_line (start 0.95 -4.1) (end 0.95 1.9) (layer B.Fab) (width 0.1))
+    (fp_line (start -0.95 -4.1) (end 0.95 -4.1) (layer B.Fab) (width 0.1))
     (fp_line (start -0.95 1.9) (end -0.95 -4.1) (layer B.Fab) (width 0.1))
-    (fp_line (start -0.95 -4.1) (end 0.95 -4.1) (layer B.Fab) (width 0.1))
-    (fp_line (start 0.95 -4.1) (end 0.95 1.9) (layer B.Fab) (width 0.1))
-    (fp_line (start 0.95 1.9) (end -0.95 1.9) (layer B.Fab) (width 0.1))
-    (fp_line (start -0.5 1.9) (end -1.27 2.7) (layer B.Fab) (width 0.1))
-    (fp_line (start -1.27 2.7) (end -1.27 3.5) (layer B.Fab) (width 0.1))
-    (fp_line (start 0.5 1.9) (end 1.27 2.7) (layer B.Fab) (width 0.1))
-    (fp_line (start 1.27 2.7) (end 1.27 3.5) (layer B.Fab) (width 0.1))
-    (fp_line (start -1.7 2.1) (end -1.7 -4.5) (layer B.SilkS) (width 0.12))
-    (fp_line (start -1.7 -4.5) (end 1.7 -4.5) (layer B.SilkS) (width 0.12))
-    (fp_line (start 1.7 -4.5) (end 1.7 2.1) (layer B.SilkS) (width 0.12))
-    (fp_line (start 1.7 2.1) (end -1.7 2.1) (layer B.SilkS) (width 0.12))
-    (fp_line (start -0.5 2.1) (end -1.27 2.5) (layer B.SilkS) (width 0.12))
-    (fp_line (start -1.27 2.5) (end -1.27 2.5) (layer B.SilkS) (width 0.12))
-    (fp_line (start 0.5 2.1) (end 1.27 2.5) (layer B.SilkS) (width 0.12))
-    (fp_line (start 1.27 2.5) (end 1.27 2.5) (layer B.SilkS) (width 0.12))
-    (fp_line (start -2.1 4.63) (end -2.1 -5.07) (layer B.CrtYd) (width 0.05))
-    (fp_line (start -2.1 -5.07) (end 2.1 -5.07) (layer B.CrtYd) (width 0.05))
-    (fp_line (start 2.1 -5.07) (end 2.1 4.63) (layer B.CrtYd) (width 0.05))
-    (fp_line (start 2.1 4.63) (end -2.1 4.63) (layer B.CrtYd) (width 0.05))
     (fp_text user %R (at 0 -0.3 180) (layer B.Fab)
       (effects (font (size 0.6 0.6) (thickness 0.09)) (justify mirror))
